Commit message: [Fix] adding pantilt plugin

File: dual_ubiquitous_display_description/urdf/pantilt/pantilt.urdf.xacro (robot description, xacro)
@@ -1,6 +1,6 @@
 <?xml version="1.0"?>
 <robot name="pantilt" xmlns:xacro="http://www.ros.org/wiki/xacro">
-  <!-- <xacro:include filename="$(find ubiquitous_display_description)/urdf/pantilt/pantilt.transmission.xacro"/>
-  <xacro:include filename="$(find ubiquitous_display_description)/urdf/pantilt/pantilt.gazebo.xacro"/> -->
+  <xacro:include filename="$(find dual_ubiquitous_display_description)/urdf/pantilt/pantilt.transmission.xacro"/>
+  <xacro:include filename="$(find dual_ubiquitous_display_description)/urdf/pantilt/pantilt.gazebo.xacro"/>
   <xacro:property name="base_to_box_height" value="0.066"/>
   <xacro:property name="box_to_proj_height" value="0.17"/>
@@ -95,4 +95,13 @@
       <dynamics damping="0.7"/>
     </joint>
+    <link name="${name}projector_plugin_optical_link" >
+    </link>
+    <joint name="${name}tilt_link_to_${name}projector_plugin_optical_link" type="fixed">
+      <origin xyz="0 -0.105 0.122 " rpy="0 -1.57 -1.57" />
+      <parent link="${name}tilt_link"/>
+      <child link="${name}projector_plugin_optical_link"/>
+    </joint>
+    <xacro:dual_ubiquitous_display_transmission name="${name}"/>
+    <xacro:pantilt_gazebo name="${name}"/>
   </xacro:macro>
 </robot>

Commit message: [Fix] replace new STL files

File: dual_ubiquitous_display_description/urdf/pantilt/pantilt.urdf.xacro (robot description, xacro)
@@ -43,8 +43,8 @@
     <link name="${name}pan_link" >
       <visual>
-        <origin xyz="0 0 -0.047" rpy="0 0 0" />
+        <origin xyz="0 0 0" rpy="0 0 0" />
         <geometry>
           <!--box size="0.07 0.085 0.065" /-->
-          <mesh filename="package://dual_ubiquitous_display_description/meshes/STL/pantilt/pantilt2_pan_link.stl" scale="0.001 0.001 0.001"/>
+          <mesh filename="package://dual_ubiquitous_display_description/meshes/STL/pantilt/pan_link.stl" scale="0.001 0.001 0.001"/>
         </geometry>
         <material name="gray"/>
@@ -62,5 +62,5 @@
       <parent link="${name}base_link"/>
       <child link="${name}pan_link"/>
-      <origin xyz="0 0 0.047" rpy="0 0 1.57" />
+      <origin xyz="0 0 0.047" rpy="0 0 0" />
       <axis xyz="0 0 1" />
       <limit lower="-2.9670" upper="2.9670" effort="41" velocity="1"/>
@@ -70,8 +70,8 @@
     <link name="${name}tilt_link" >
       <visual>
-        <origin xyz=" -0.250 0 0.118" rpy="0 0 0" />
+        <origin xyz=" 0 0 0" rpy="1.57 0 0" />
         <geometry>
           <!--box size="0.07 0.085 0.065" /-->
-          <mesh filename="package://dual_ubiquitous_display_description/meshes/STL/pantilt/pantilt2_tilt_link.stl" scale="0.001 0.001 0.001"/>
+          <mesh filename="package://dual_ubiquitous_display_description/meshes/STL/pantilt/tilt_link.stl" scale="0.001 0.001 0.001"/>
         </geometry>
         <material name="gray"/>
@@ -89,5 +89,5 @@
       <parent link="${name}pan_link"/>
       <child link="${name}tilt_link"/>
-      <origin xyz="0 0.118 ${0.250-0.047}" rpy="1.57 -1.57 0" />
+      <origin xyz="0.093 0 0.195" rpy="0 -1.57 0" />
       <axis xyz="0 0 1" />
       <limit lower="-1.3" upper="1.3" effort="10" velocity="1"/>
@@ -98,5 +98,5 @@
     </link>
     <joint name="${name}tilt_link_to_${name}projector_plugin_optical_link" type="fixed">
-      <origin xyz="0 -0.105 0.122 " rpy="0 -1.57 -1.57" />
+      <origin xyz="0 0 0.093 " rpy="-1.57 3.14 0" />
       <parent link="${name}tilt_link"/>
       <child link="${name}projector_plugin_optical_link"/>
