Commit message: [Fix] adjust pan angle offset

File: dual_ubiquitous_display_description/robots/dual_ubiquitous_display_for_gazebo.urdf.xacro (robot description, xacro)
@@ -5,6 +5,6 @@
   <xacro:include filename="$(find dual_ubiquitous_display_description)/urdf/pantilt/pantilt.urdf.xacro"/>
   <xacro:include filename="$(find dual_ubiquitous_display_description)/urdf/sensor/lrf/hokuyo_utm30lx.urdf.xacro"/>
-  <xacro:pantilt_model name="pantilt1_" parent="body_link" pos="0.18" offset="0.392699"/>
-  <xacro:pantilt_model name="pantilt2_" parent="body_link" pos="-0.18" offset="0.392699"/>
+  <xacro:pantilt_model name="pantilt1_" parent="body_link" pos="0.18" offset="0.0"/>
+  <xacro:pantilt_model name="pantilt2_" parent="body_link" pos="-0.18" offset="0.0"/>
   <!--xacro:hokuyo_utm30lx_model name="front_laser" parent="base_link" pos="0.261" ang="0"/>
   <xacro:hokuyo_utm30lx_model name="rear_laser" parent="base_link" pos="-0.261" ang="3.14"/-->

File: dual_ubiquitous_display_description/urdf/pantilt/pantilt.urdf.xacro (robot description, xacro)
@@ -17,5 +17,5 @@
     <color rgba="0.7 0.7 0.7 1.0" />
   </material>
-  <xacro:macro name="pantilt_model" params="name parent pos">
+  <xacro:macro name="pantilt_model" params="name parent pos offset">
     <link name="${name}base_link" >
       <visual>
@@ -62,5 +62,5 @@
       <parent link="${name}base_link"/>
       <child link="${name}pan_link"/>
-      <origin xyz="0 0 0.047" rpy="0 0 0" />
+      <origin xyz="0 0 0.047" rpy="0 0 ${-offset}" />
       <axis xyz="0 0 1" />
       <limit lower="-2.9670" upper="2.9670" effort="41" velocity="1"/>
