Commit message: [Edit] base ~ body parameters

File: dual_ubiquitous_display_description/robots/dual_ubiquitous_display.urdf.xacro (robot description, xacro)
@@ -3,5 +3,7 @@
   <xacro:include filename="$(find dual_ubiquitous_display_description)/urdf/body/body.urdf.xacro"/>
   <xacro:include filename="$(find dual_ubiquitous_display_description)/urdf/youbot/youbot_base_only.urdf.xacro"/>
+  <xacro:include filename="$(find dual_ubiquitous_display_description)/urdf/pantilt/pantilt.urdf.xacro"/>
   <!-- <xacro:include filename="$(find dual_ubiquitous_display_description)/urdf/sensor/lrf/hokuyo_utm30lx.urdf.xacro"/> -->
+  <xacro:pantilt_model name="pantilt2_" parent="body_link"/>
   <!-- <xacro:hokuyo_utm30lx_model name="front_laser" parent="front_laser_adjuster_link" /> -->
   <!-- <xacro:hokuyo_utm30lx_model name="rear_laser" parent="rear_laser_adjuster_link" /> -->

File: dual_ubiquitous_display_description/urdf/body/body.urdf.xacro (robot description, xacro)
@@ -3,5 +3,5 @@
   <!-- <xacro:include filename="$(find ubiquitous_display_description)/urdf/body/body.gazebo.xacro"/> -->
   <joint name="base_link_to_body_link" type="fixed">
-    <origin xyz="0 0 0" rpy="0 0 0" />
+    <origin xyz="0 0 0.349" rpy="0 0 0" />
     <parent link="base_link"/>
     <child link="body_link"/>
@@ -13,5 +13,5 @@
         <mesh filename="package://dual_ubiquitous_display_description/meshes/STL/body/dud_body.stl" scale="0.001 0.001 0.001"/>
       </geometry>
-      <origin xyz="0.0 0.0 0.0"/>
+      <origin xyz="0.0 0.0 -0.349"/>
       <material name="white" />
     </visual>

Commit message: [Add] dual pantilt link

File: dual_ubiquitous_display_description/robots/dual_ubiquitous_display.urdf.xacro (robot description, xacro)
@@ -5,5 +5,6 @@
   <xacro:include filename="$(find dual_ubiquitous_display_description)/urdf/pantilt/pantilt.urdf.xacro"/>
   <!-- <xacro:include filename="$(find dual_ubiquitous_display_description)/urdf/sensor/lrf/hokuyo_utm30lx.urdf.xacro"/> -->
-  <xacro:pantilt_model name="pantilt2_" parent="body_link"/>
+  <xacro:pantilt_model name="pantilt1_" parent="body_link" pos="0.18"/>
+  <xacro:pantilt_model name="pantilt2_" parent="body_link" pos="-0.18"/>
   <!-- <xacro:hokuyo_utm30lx_model name="front_laser" parent="front_laser_adjuster_link" /> -->
   <!-- <xacro:hokuyo_utm30lx_model name="rear_laser" parent="rear_laser_adjuster_link" /> -->

File: dual_ubiquitous_display_description/urdf/pantilt/pantilt.urdf.xacro (robot description, xacro)
@@ -17,5 +17,5 @@
     <color rgba="0.7 0.7 0.7 1.0" />
   </material>
-  <xacro:macro name="pantilt_model" params="name parent">
+  <xacro:macro name="pantilt_model" params="name parent pos">
     <link name="${name}base_link" >
       <visual>
@@ -37,8 +37,62 @@
     </link>
     <joint name="${parent}_to_${name}base_link" type="fixed">
-      <origin xyz="0 0 0.372 " rpy="0 0 0" />
+      <origin xyz="${pos} 0 0.372 " rpy="0 0 0" />
       <parent link="${parent}"/>
       <child link="${name}base_link"/>
     </joint>
+    <link name="${name}pan_link" >
+      <visual>
+        <origin xyz="0 0 -0.047" rpy="0 0 0" />
+        <geometry>
+          <!--box size="0.07 0.085 0.065" /-->
+          <mesh filename="package://dual_ubiquitous_display_description/meshes/STL/pantilt/pantilt2_pan_link.stl" scale="0.001 0.001 0.001"/>
+        </geometry>
+        <material name="gray"/>
+      </visual>
+     <inertial>
+       <origin xyz="0 0 ${base_to_box_height/2}" rpy="0 0 0"/>
+       <mass value="0.78"/>
+       <inertia
+	    ixx="0.00190" ixy="0.0" ixz="0.0"
+	    iyy="0.00202" iyz="0.0"
+	    izz="0.00152"/>
+     </inertial>
+    </link>
+    <joint name="${name}pan_joint" type="revolute">
+      <parent link="${name}base_link"/>
+      <child link="${name}pan_link"/>
+      <origin xyz="0 0 0.047" rpy="0 0 1.57" />
+      <axis xyz="0 0 1" />
+      <limit lower="-2.9670" upper="2.9670" effort="41" velocity="1"/>
+      <!--<safety_controller k_velocity="10" k_position="15" soft_lower_limit="-2.0" soft_upper_limit="0.5" />-->
+      <dynamics damping="0.7"/>
+    </joint>
+    <link name="${name}tilt_link" >
+      <visual>
+        <origin xyz=" -0.250 0 0.118" rpy="0 0 0" />
+        <geometry>
+          <!--box size="0.07 0.085 0.065" /-->
+          <mesh filename="package://dual_ubiquitous_display_description/meshes/STL/pantilt/pantilt2_tilt_link.stl" scale="0.001 0.001 0.001"/>
+        </geometry>
+        <material name="gray"/>
+      </visual>
+     <inertial>
+       <origin xyz="-0.250 0 0.118" rpy="0 0 0"/>
+       <mass value="0.78"/>
+       <inertia
+      ixx="0.00190" ixy="0.0" ixz="0.0"
+      iyy="0.00202" iyz="0.0"
+      izz="0.00152"/>
+     </inertial>
+    </link>
+    <joint name="${name}tilt_joint" type="revolute">
+      <parent link="${name}pan_link"/>
+      <child link="${name}tilt_link"/>
+      <origin xyz="0 0.118 ${0.250-0.047}" rpy="1.57 -1.57 0" />
+      <axis xyz="0 0 1" />
+      <limit lower="-1.3" upper="1.3" effort="10" velocity="1"/>
+      <!--<safety_controller k_velocity="10" k_position="15" soft_lower_limit="-2.0" soft_upper_limit="0.5" />-->
+      <dynamics damping="0.7"/>
+    </joint>
   </xacro:macro>
 </robot>

Commit message: [[Edit] lrf plugin

File: dual_ubiquitous_display_description/robots/dual_ubiquitous_display.urdf.xacro (robot description, xacro)
@@ -4,9 +4,9 @@
   <xacro:include filename="$(find dual_ubiquitous_display_description)/urdf/youbot/youbot_base_only.urdf.xacro"/>
   <xacro:include filename="$(find dual_ubiquitous_display_description)/urdf/pantilt/pantilt.urdf.xacro"/>
-  <!-- <xacro:include filename="$(find dual_ubiquitous_display_description)/urdf/sensor/lrf/hokuyo_utm30lx.urdf.xacro"/> -->
+  <xacro:include filename="$(find dual_ubiquitous_display_description)/urdf/sensor/lrf/hokuyo_utm30lx.urdf.xacro"/>
   <xacro:pantilt_model name="pantilt1_" parent="body_link" pos="0.18"/>
   <xacro:pantilt_model name="pantilt2_" parent="body_link" pos="-0.18"/>
-  <!-- <xacro:hokuyo_utm30lx_model name="front_laser" parent="front_laser_adjuster_link" /> -->
-  <!-- <xacro:hokuyo_utm30lx_model name="rear_laser" parent="rear_laser_adjuster_link" /> -->
+  <xacro:hokuyo_utm30lx_model name="front_laser" parent="base_link" pos="0.261" ang="0"/>
+  <xacro:hokuyo_utm30lx_model name="rear_laser" parent="base_link" pos="-0.261" ang="3.14"/>
   <!-- =============== Gazebo =============== -->
   <gazebo>

File: dual_ubiquitous_display_description/urdf/sensor/lrf/hokuyo_utm30lx.urdf.xacro (robot description, xacro)
@@ -3,8 +3,8 @@
     <xacro:include filename="$(find ubiquitous_display_description)/urdf/sensor/lrf/hokuyo_utm30lx.gazebo.xacro"/>
     <xacro:property name="M_PI" value="3.1415926535897931" />
-    <xacro:macro name="hokuyo_utm30lx_model" params="name parent">
+    <xacro:macro name="hokuyo_utm30lx_model" params="name parent pos ang">
       <joint name="${name}_joint" type="fixed">
         <!--xacro:insert_block name="origin" /-->
-        <origin xyz="-0.029 0 0.067" rpy="0 0 0"/>
+        <origin xyz="${pos} 0 0.178" rpy="0 0 ${ang}"/>
         <parent link="${parent}"/>
         <child link="${name}_frame"/>

Commit message: [Fix] D-UD urdf model (using new top plate)

File: dual_ubiquitous_display_description/robots/dual_ubiquitous_display.urdf.xacro (robot description, xacro)
@@ -5,8 +5,8 @@
   <xacro:include filename="$(find dual_ubiquitous_display_description)/urdf/pantilt/pantilt.urdf.xacro"/>
   <xacro:include filename="$(find dual_ubiquitous_display_description)/urdf/sensor/lrf/hokuyo_utm30lx.urdf.xacro"/>
-  <xacro:pantilt_model name="pantilt1_" parent="body_link" pos="0.18" offset="0.392699"/>
-  <xacro:pantilt_model name="pantilt2_" parent="body_link" pos="-0.18" offset="0.392699"/>
-  <!--xacro:hokuyo_utm30lx_model name="front_laser" parent="base_link" pos="0.261" ang="0"/>
-  <xacro:hokuyo_utm30lx_model name="rear_laser" parent="base_link" pos="-0.261" ang="3.14"/-->
+  <xacro:pantilt_model name="pantilt1_" parent="body_link" pos="0.225" offset="0"/>  <!-- offset="0.392699" -->
+  <xacro:pantilt_model name="pantilt2_" parent="body_link" pos="-0.225" offset="0"/>  <!-- offset="0.392699" -->
+  <xacro:hokuyo_utm30lx_model name="front_laser" parent="base_link" pos="0.261" ang="0"/>
+  <xacro:hokuyo_utm30lx_model name="rear_laser" parent="base_link" pos="-0.261" ang="3.14"/>
   <!-- =============== Gazebo =============== -->
   <gazebo>

File: dual_ubiquitous_display_description/urdf/body/body.gazebo.xacro (robot description, xacro)
@@ -1,23 +1,9 @@
 <?xml version="1.0"?>
 <robot name="body_gazebo" xmlns:xacro="http://www.ros.org/wiki/xacro">
-<xacro:macro name="plate_template_gazebo" params="name">
-  <gazebo reference="${name}_plate_link">
+<xacro:macro name="plate_template_gazebo">
+  <gazebo reference="body_link">
     <mu1>0.2</mu1>
     <mu2>0.2</mu2>
-    <!--material>Gazebo/LightGrey</material-->
-  </gazebo>
-</xacro:macro>
-<xacro:macro name="pillar_template_gazebo" params="name">
-  <gazebo reference="${name}_pillars_link">
-    <mu1>0.2</mu1>
-    <mu2>0.2</mu2>
-    <material>Gazebo/Black</material>
-  </gazebo>
-</xacro:macro>
-<xacro:macro name="laser_adjuster_template_gazebo" params="name">
-  <gazebo reference="${name}_laser_adjuster_link">
-    <mu1>0.2</mu1>
-    <mu2>0.2</mu2>
-    <material>Gazebo/White</material>
+    <material>Gazebo/Grey</material>
   </gazebo>
 </xacro:macro>

File: dual_ubiquitous_display_description/urdf/body/body.urdf.xacro (robot description, xacro)
@@ -1,7 +1,7 @@
 <?xml version="1.0"?>
 <robot name="body" xmlns:xacro="http://www.ros.org/wiki/xacro">
-  <!-- <xacro:include filename="$(find ubiquitous_display_description)/urdf/body/body.gazebo.xacro"/> -->
+  <xacro:include filename="$(find dual_ubiquitous_display_description)/urdf/body/body.gazebo.xacro"/>
   <joint name="base_link_to_body_link" type="fixed">
-    <origin xyz="0 0 0.349" rpy="0 0 0" />
+    <origin xyz="0 0.0 0.349" rpy="0 0 0" />
     <parent link="base_link"/>
     <child link="body_link"/>
@@ -11,9 +11,10 @@
       <geometry>
         <!-- <box size="0.5 0.5 1.0"/> -->
-        <mesh filename="package://dual_ubiquitous_display_description/meshes/STL/body/dud_body.stl" scale="0.001 0.001 0.001"/>
+        <mesh filename="package://dual_ubiquitous_display_description/meshes/STL/body/complete.stl" scale="0.001 0.001 0.001"/>
       </geometry>
-      <origin xyz="0.0 0.0 -0.349"/>
-      <material name="white" />
+      <origin xyz="0.03865 -0.15 -0.349"/>
+      <material name="gray" />
     </visual>
   </link>
+  <xacro:plate_template_gazebo />
 </robot>

File: dual_ubiquitous_display_description/urdf/pantilt/pantilt.gazebo.xacro (robot description, xacro)
@@ -5,15 +5,15 @@
     <mu1>0.2</mu1>
     <mu2>0.2</mu2>
-    <material>Gazebo/LightGrey</material>
+    <material>Gazebo/Grey</material>
   </gazebo>
   <gazebo reference="${name}tilt_link">
     <mu1>0.2</mu1>
     <mu2>0.2</mu2>
-    <material>Gazebo/LightGrey</material>
+    <material>Gazebo/Grey</material>
   </gazebo>
   <gazebo reference="${name}pan_link">
     <mu1>0.2</mu1>
     <mu2>0.2</mu2>
-    <material>Gazebo/LightGrey</material>
+    <material>Gazebo/Grey</material>
   </gazebo>
   <gazebo reference="${name}projector_plugin_optical_link">

File: dual_ubiquitous_display_description/urdf/sensor/lrf/hokuyo_utm30lx.urdf.xacro (robot description, xacro)
@@ -1,5 +1,5 @@
 <?xml version="1.0"?>
 <robot xmlns:xacro="http://ros.org/wiki/xacro">
-    <xacro:include filename="$(find ubiquitous_display_description)/urdf/sensor/lrf/hokuyo_utm30lx.gazebo.xacro"/>
+    <xacro:include filename="$(find dual_ubiquitous_display_description)/urdf/sensor/lrf/hokuyo_utm30lx.gazebo.xacro"/>
     <xacro:property name="M_PI" value="3.1415926535897931" />
     <xacro:macro name="hokuyo_utm30lx_model" params="name parent pos ang">
@@ -11,4 +11,10 @@
       </joint>
       <link name="${name}_frame">
+        <visual>
+          <origin xyz="0 0 0" rpy="0 0 0" />
+          <geometry>
+            <mesh filename="package://ubiquitous_display_description/meshes/DAE/hokuyo_utm_30lx.dae"/>
+          </geometry>
+        </visual>
         <inertial>
           <mass value="0.270" />
@@ -16,16 +22,10 @@
           <inertia ixx="2.632e-4" ixy="0" ixz="0" iyy="2.632e-4" iyz="0" izz="1.62e-4" />
         </inertial>
-        <visual>
-          <origin xyz="0 0 0" rpy="0 0 0" />
-          <geometry>
-          <mesh filename="package://ubiquitous_display_description/meshes/DAE/hokuyo_utm_30lx.dae"/>
-        </geometry>
-        </visual>
         <collision>
           <origin xyz="0 0 -0.0115" rpy="0 0 0" />
           <geometry>
-          <box size="0.058 0.058 0.087" />
-          <!--<mesh filename="package://hector_sensors_description/meshes/hokuyo_utm30lx/hokuyo_utm_30lx.stl"/>-->
-        </geometry>
+            <box size="0.058 0.058 0.087" />
+            <!--<mesh filename="package://hector_sensors_description/meshes/hokuyo_utm30lx/hokuyo_utm_30lx.stl"/>-->
+          </geometry>
         </collision>
       </link>
